Commit message: Add missing M_PI property

File: tiago_description/robots/tiago_steel.urdf.xacro (robot description, xacro)
@@ -9,4 +9,5 @@
 <robot  xmlns:xacro="http://www.ros.org/wiki/xacro"
         name="tiago" >
+  <xacro:property name="M_PI" value="3.141592653589793" />
   <!-- The following included files set up definitions of parts of the robot body -->
   <!-- Base -->
